Commit message: style fix

File: src/multibot_model/description/robot/wheele_core.xacro (robot description, xacro)
@@ -42,4 +42,6 @@
     <!-- MACRO FOR THE WHEELS -->
     <xacro:macro name="wheel" params="prefix reflect_x reflect_y">
+        <xacro:property name="pose_wheel" value="0 0 0"/>
+        <xacro:property name="orientation_wheel" value="0 0 ${pi/2 + reflect_y * pi/2}"/>
         <joint name="base_to_${prefix}_wheel" type="continuous">
             <parent link="chassis"/>
@@ -53,5 +55,5 @@
                     <cylinder radius="${wheel_radius}" length="${wheel_thickness}"/>
                 </geometry>
-                <origin xyz="0 0 0" rpy="0 0 ${pi/2 + reflect_y * pi/2}"/>
+                <origin xyz="0 0 0" rpy="${orientation_wheel}"/>
                 <material name="white"/>
             </visual>
@@ -60,8 +62,8 @@
                     <cylinder radius="${wheel_radius}" length="${wheel_thickness}"/>
                 </geometry>
-                <origin xyz="0 0 0" rpy="0 0 ${pi/2 + reflect_y * pi/2}"/>
+                <origin xyz="0 0 0" rpy="${orientation_wheel}"/>
             </collision>
             <xacro:inertial_cylinder mass="${wheel_mass}" length="${wheel_thickness}" radius="${wheel_radius}">
-                <origin xyz="0 0 0" rpy="0 0 0"/>
+                <origin xyz="0 0 0" rpy="${orientation_wheel}"/>
             </xacro:inertial_cylinder>
         </link>
@@ -71,4 +73,5 @@
     </xacro:macro>
     <!-- BASE LINK -->
+    <link name="base_link"/>
     <link name="base_footprint"/>
     <!-- BASE_FOOTPRINT LINK -->
@@ -78,5 +81,4 @@
         <origin xyz="0 0 0" rpy="0 0 0"/>
     </joint>
-    <link name="base_link"/>
     <!-- CHASSIS LINK -->
     <joint name="chassis_joint" type="fixed">
@@ -120,5 +122,4 @@
     </link>
     <!-- Swivel -->
-    <!--                xyz="${wheelbase_length/2} 0 ${caster_wheel_radius*2}"-->
     <joint name="caster_yaw_joint" type="continuous">
         <parent link="chassis"/>
