Commit message: fix control

File: src/multibot_model/description/robot/macros_gazebo_control.xacro (robot description, xacro)
@@ -1,15 +1,20 @@
 <?xml version="1.0"?>
 <robot xmlns:xacro="http://www.ros.org/wiki/xacro" >
-<!--    <gazebo>-->
-<!--        &lt;!&ndash; Differential Drive Plugin &ndash;&gt;-->
-<!--        <plugin filename="gz-sim-diff-drive-system"-->
-<!--                name="gz::sim::systems::DiffDrive">-->
-<!--            &lt;!&ndash; Match the joint names from wheele_core.xacro &ndash;&gt;-->
-<!--            <left_joint>left_wheel_joint</left_joint>-->
-<!--            <right_joint>right_wheel_joint</right_joint>-->
-<!--            &lt;!&ndash; Match actual robot dimensions &ndash;&gt;-->
-<!--            <wheel_separation>${0.3 + 0.085}</wheel_separation>  &lt;!&ndash; track width &ndash;&gt;-->
-<!--            <wheel_radius>0.07</wheel_radius>-->
-<!--            &lt;!&ndash; Control parameters &ndash;&gt;-->
+    <gazebo>
+        <!-- Differential Drive Plugin -->
+        <!--official documentation-->
+        <!--https://gazebosim.org/api/sim/8/classgz_1_1sim_1_1systems_1_1DiffDrive.html-->
+        <!--this Plugin will publish those topics-->
+        <!--/model/bot1/odometry    publisher   gz.msgs.Odometry-->
+        <!--/model/bot1/tf          publisher   gz.msgs.Pose_V      publish the transform from frame_id to child_frame_id-->
+        <!--/model/bot1/cmd_vel     subscriber  gz.msgs.Twist    -->
+        <!--/model/bot1/enable      subscriber  gz.msgs.Boolean-->
+        <plugin filename="gz-sim-diff-drive-system"
+                name="gz::sim::systems::DiffDrive">
+            <left_joint>chassis_rear_left_wheel</left_joint>
+            <right_joint>chassis_rear_right_wheel</right_joint>
+            <wheel_separation>${chassis_width + wheel_thickness}</wheel_separation>  <!-- track width -->
+            <wheel_radius>${wheel_radius}</wheel_radius>
+            <!-- Control parameters -->
 <!--            <odom_publish_frequency>50</odom_publish_frequency>-->
 <!--            <max_linear_acceleration>1.0</max_linear_acceleration>-->
@@ -21,19 +26,22 @@
 <!--            <max_angular_velocity>1.0</max_angular_velocity>-->
 <!--            <min_angular_velocity>-1.0</min_angular_velocity>-->
-<!--            &lt;!&ndash; Topic configuration &ndash;&gt;-->
+            <!-- Topic configuration -->
 <!--            <topic>cmd_vel</topic>-->
 <!--            <odom_topic>odom</odom_topic>-->
-<!--            <frame_id>odom</frame_id>-->
-<!--            <child_frame_id>base_footprint</child_frame_id>-->
-<!--        </plugin>-->
-<!--        &lt;!&ndash; Joint State Publisher &ndash;&gt;-->
+<!--            @todo tbd if neccessary-->
+            <frame_id>odom</frame_id>
+            <child_frame_id>base_footprint</child_frame_id>
+        </plugin>
+        <!-- Joint State Publisher -->
+        <!--official documentation-->
+        <!--https://gazebosim.org/api/sim/8/classgz_1_1sim_1_1systems_1_1JointStatePublisher.html-->
 <!--        <plugin filename="gz-sim-joint-state-publisher-system"-->
 <!--                name="gz::sim::systems::JointStatePublisher">-->
-<!--            <joint_name>left_wheel_joint</joint_name>-->
-<!--            <joint_name>right_wheel_joint</joint_name>-->
-<!--            <joint_name>caster_yaw_joint</joint_name>-->
-<!--            <joint_name>caster_wheel_joint</joint_name>-->
+<!--&lt;!&ndash;            <joint_name>left_wheel_joint</joint_name>&ndash;&gt;-->
+<!--&lt;!&ndash;            <joint_name>right_wheel_joint</joint_name>&ndash;&gt;-->
+<!--&lt;!&ndash;            <joint_name>caster_yaw_joint</joint_name>&ndash;&gt;-->
+<!--&lt;!&ndash;            <joint_name>caster_wheel_joint</joint_name>&ndash;&gt;-->
 <!--        </plugin>-->
-<!--        &lt;!&ndash; Pose Publisher (optional, for debugging) &ndash;&gt;-->
+        <!-- Pose Publisher (optional, for debugging) -->
 <!--        <plugin filename="gz-sim-pose-publisher-system"-->
 <!--                name="gz::sim::systems::PosePublisher">-->
@@ -45,4 +53,4 @@
 <!--            <update_frequency>50</update_frequency>-->
 <!--        </plugin>-->
-<!--    </gazebo>-->
+    </gazebo>
 </robot>

File: src/multibot_model/description/robot/model.urdf.xacro (robot description, xacro)
@@ -1,4 +1,4 @@
 <?xml version="1.0"?>
-<robot xmlns:xacro="http://www.ros.org/wiki/xacro"  name="bot1">
+<robot xmlns:xacro="http://www.ros.org/wiki/xacro"  name="$(env ROBOT_NAME)">
     <xacro:include filename="wheele_core.xacro" />
     <xacro:include filename="macros_gazebo_control.xacro" />

File: src/multibot_model/description/robot/tmp.urdf (robot description, URDF)
Before this commit: robot bot1, 7 links, 6 joints
Joints:
- removed joint base_to_rear_left_wheel
- removed joint base_to_rear_right_wheel
- added joint chassis_rear_left_wheel: type continuous, parent chassis, child rear_left_wheel, origin xyz=-0.15 -0.1925 0 rpy=0 1.5707963267948966 1.5707963267948966, axis 0 1 0
- added joint chassis_rear_right_wheel: type continuous, parent chassis, child rear_right_wheel, origin xyz=-0.15 0.1925 0 rpy=0 1.5707963267948966 1.5707963267948966, axis 0 1 0

File: src/multibot_model/description/robot/wheele_core.xacro (robot description, xacro)
@@ -44,9 +44,9 @@
         <xacro:property name="pose_wheel" value="0 0 0"/>
         <xacro:property name="orientation_wheel" value="0 0 ${pi/2 + reflect_y * pi/2}"/>
-        <joint name="base_to_${prefix}_wheel" type="continuous">
+        <joint name="chassis_${prefix}_wheel" type="continuous">
             <parent link="chassis"/>
             <child link="${prefix}_wheel"/>
             <origin xyz="${reflect_x * wheelbase_length/2} ${reflect_y * track/2} 0" rpy="0 ${pi/2} ${pi/2}"/>
-            <axis xyz="0 1 0"/>
+            <axis xyz="0 0 1"/>
         </joint>
         <link name="${prefix}_wheel">
@@ -160,6 +160,6 @@
     </joint>
     <gazebo reference="caster">
-        <mu1>0.6</mu1>
-        <mu2>0.6</mu2>
+        <mu1>0.01</mu1>
+        <mu2>0.01</mu2>
     </gazebo>
 </robot>

Commit message: fix tf tree

File: src/multibot_model/description/robot/macros_gazebo_control.xacro (robot description, xacro)
@@ -36,21 +36,21 @@
         <!--official documentation-->
         <!--https://gazebosim.org/api/sim/8/classgz_1_1sim_1_1systems_1_1JointStatePublisher.html-->
-<!--        <plugin filename="gz-sim-joint-state-publisher-system"-->
-<!--                name="gz::sim::systems::JointStatePublisher">-->
-<!--&lt;!&ndash;            <joint_name>left_wheel_joint</joint_name>&ndash;&gt;-->
-<!--&lt;!&ndash;            <joint_name>right_wheel_joint</joint_name>&ndash;&gt;-->
-<!--&lt;!&ndash;            <joint_name>caster_yaw_joint</joint_name>&ndash;&gt;-->
-<!--&lt;!&ndash;            <joint_name>caster_wheel_joint</joint_name>&ndash;&gt;-->
-<!--        </plugin>-->
+        <plugin filename="gz-sim-joint-state-publisher-system"
+                name="gz::sim::systems::JointStatePublisher">
+            <joint_name>chassis_rear_left_wheel</joint_name>
+            <joint_name>chassis_rear_right_wheel</joint_name>
+            <joint_name>caster_yaw_joint</joint_name>
+            <joint_name>caster_wheel_joint</joint_name>
+        </plugin>
         <!-- Pose Publisher (optional, for debugging) -->
-<!--        <plugin filename="gz-sim-pose-publisher-system"-->
-<!--                name="gz::sim::systems::PosePublisher">-->
-<!--            <publish_link_pose>true</publish_link_pose>-->
-<!--            <publish_collision_pose>false</publish_collision_pose>-->
-<!--            <publish_visual_pose>false</publish_visual_pose>-->
-<!--            <publish_nested_model_pose>false</publish_nested_model_pose>-->
-<!--            <use_pose_vector_msg>true</use_pose_vector_msg>-->
-<!--            <update_frequency>50</update_frequency>-->
-<!--        </plugin>-->
+        <plugin filename="gz-sim-pose-publisher-system"
+                name="gz::sim::systems::PosePublisher">
+            <publish_link_pose>true</publish_link_pose>
+            <publish_collision_pose>false</publish_collision_pose>
+            <publish_visual_pose>false</publish_visual_pose>
+            <publish_nested_model_pose>false</publish_nested_model_pose>
+            <use_pose_vector_msg>true</use_pose_vector_msg>
+            <update_frequency>50</update_frequency>
+        </plugin>
     </gazebo>
 </robot>

File: src/multibot_model/description/robot/tmp.urdf (robot description, URDF)
Before this commit: robot bot1, 7 links, 6 joints
Joints:
- joint base_footprint_joint: child base_footprint -> base_link; parent base_link -> base_footprint
- joint chassis_rear_left_wheel: axis 0 1 0 -> 0 0 1
- joint chassis_rear_right_wheel: axis 0 1 0 -> 0 0 1

File: src/multibot_model/description/robot/wheele_core.xacro (robot description, xacro)
@@ -77,6 +77,6 @@
     <!-- BASE_FOOTPRINT LINK -->
     <joint name="base_footprint_joint" type="fixed">
-        <child link="base_footprint"/>
-        <parent link="base_link"/>
+        <parent link="base_footprint"/>
+        <child link="base_link"/>
         <origin xyz="0 0 0" rpy="0 0 0"/>
     </joint>
