Commit message: update noise bridge

File: src/multibot_model/description/robot/model.urdf.xacro (robot description, xacro)
@@ -3,7 +3,7 @@
     <xacro:include filename="wheele_core.xacro" />
     <xacro:include filename="macros_gazebo_control.xacro" />
-<!--    <xacro:include filename="gazebo_sensors/lidar.xacro" />-->
-<!--    <xacro:include filename="gazebo_sensors/gps.xacro" />-->
-<!--    <xacro:include filename="gazebo_sensors/imu.xacro" />-->
+    <xacro:include filename="gazebo_sensors/lidar.xacro" />
+    <xacro:include filename="gazebo_sensors/gps.xacro" />
+    <xacro:include filename="gazebo_sensors/imu.xacro" />
 <!--    <xacro:include filename="gazebo_sensors/collision_sensor.xacro" />-->
 <!--    <xacro:include filename="gazebo_sensors/camera.xacro" />-->

File: src/multibot_model/description/robot/tmp.urdf (robot description, URDF)
Before this commit: robot bot1, 7 links, 6 joints
Links:
- added link gps, mass 0.1; collision cylinder length=0.02 radius=0.01; visual cylinder length=0.02 radius=0.01
- added link imu, mass 0.001; collision box size=0.01 0.01 0.005; visual box size=0.01 0.01 0.005
- added link laser, mass 0.1; collision cylinder length=0.04 radius=0.019; visual cylinder length=0.04 radius=0.019
Joints:
- added joint gps_joint: type fixed, parent chassis, child gps, origin xyz=-0.185 -0.09999999999999999 0.30000000000000004 rpy=0 0 0
- added joint imu_joint: type fixed, parent chassis, child imu, origin xyz=0.03499999999999999 0.0 0.21000000000000002 rpy=0 0 0
- added joint laser_joint: type fixed, parent chassis, child laser, origin xyz=0.18999999999999997 -0.10099999999999999 0.22 rpy=0 0 0
